Commit message: 完成要求但识别不稳

File: avs_ws/src/avs_rescue_sim/urdf/rescue_rover.urdf (robot description, URDF)
Before this commit: robot rescue_rover, 8 links, 7 joints
Links:
- link pusher_link: geometry collision box size=0.14 0.28 0.10; collision box size=0.18 0.055 0.10
Joints:
- joint camera_joint: axis (none) -> 0 0 1; limit (none) -> lower=-1.95 upper=1.95 effort=2 velocity=1.2; type fixed -> revolute

Commit message: 答辩

File: avs_ws/src/avs_rescue_sim/urdf/rescue_rover.urdf (robot description, URDF)
Before this commit: robot rescue_rover, 8 links, 7 joints
Links:
- link base_link: geometry collision box size=0.42 0.24 0.14; visual box size=0.04 0.05 0.006
- link camera_link: geometry visual box size=0.06 0.09 0.06; visual cylinder length=0.003 radius=0.018
